Commit message: 3d rigid body - Works!

File: ocs2_object_manipulation_ros/urdf/object.urdf (robot description, URDF)
Before this commit: robot cartpole, 5 links, 4 joints
Links:
- added link object_target, mass 2; collision box size=0.5 0.5 0.5; visual box size=0.5 0.5 0.5
- added link prismatic_x_target, mass 0.001
- added link prismatic_y_target, mass 0.001
Joints:
- added joint theta_target: type continuous, parent prismatic_y_target, child object_target, origin xyz=0.0 0.0 0 rpy=0.0 0.0 0.0, axis 0 0 1
- added joint x_target: type prismatic, parent ground, child prismatic_x_target, origin xyz=0.0 0.0 0.0, axis 1 0 0, limit lower=-150 upper=150 effort=100000.0 velocity=50
- added joint y_target: type prismatic, parent prismatic_x_target, child prismatic_y_target, origin xyz=0.0 0.0 0.0, axis 0 1 0, limit lower=-150 upper=150 effort=100000.0 velocity=50

Commit message: add rviz visualizer

File: ocs2_object_manipulation_ros/urdf/object.urdf (robot description, URDF)
Before this commit: robot object, 8 links, 7 joints
Links:
- link ground: geometry 
